Commit message: Update robot description sdf

File: src/polebot_land/urdf/gazebo_plugin.xacro (robot description, xacro)
@@ -9,5 +9,5 @@
     <plugin name="ignition::gazebo::systems::Imu" filename="libignition-gazebo-imu-system.so" />
     <plugin filename="ign_ros2_control-system" name="ign_ros2_control::IgnitionROS2ControlPlugin">
-      <parameters>$(find robotpadi)/config/diff_drive_controller.yaml</parameters>
+      <parameters>$(find polebot_land)/config/diff_drive_controller.yaml</parameters>
     </plugin>
   </gazebo> -->
@@ -17,5 +17,5 @@
           <namespace>$(arg namespace)</namespace>
       </ros>
-      <parameters>$(find robotpadi)/config/diff_drive_controller.yaml</parameters>
+      <parameters>$(find polebot_land)/config/diff_drive_controller.yaml</parameters>
       </plugin>
   </gazebo>

File: src/polebot_land/urdf/main.xacro (robot description, xacro)
@@ -1,5 +1,5 @@
 <?xml version="1.0"?>
 <robot xmlns:xacro="http://www.ros.org/wiki/xacro" name="robot_padi">
-    <xacro:include filename="robot_padi.xacro"/>
+    <xacro:include filename="polebot_land.xacro"/>
     <xacro:include filename="ros2_control.xacro"/>
     <!-- <xacro:include filename="gazebo_plugin.xacro"/> -->

File: src/polebot_land/urdf/polebot_land.xacro (robot description, xacro)
@@ -4,6 +4,6 @@
      For more information, please see http://wiki.ros.org/sw_urdf_exporter -->
 <robot xmlns:xacro="http://www.ros.org/wiki/xacro">
-  <xacro:property name="mesh_path" value="$(find robotpadi)/meshes"/>
-  <xacro:include filename="$(find robotpadi)/urdf/imu.xacro" />
+  <xacro:property name="mesh_path" value="$(find polebot_land)/meshes"/>
+  <xacro:include filename="$(find polebot_land)/urdf/imu.xacro" />
   <link name="base_footprint"/>
   <joint name="base_footprint_to_base_link_joint" type="fixed">
@@ -359,5 +359,5 @@
   <plugin name="gazebo_ros_odometry" filename="libgazebo_ros_odometry.so">
     <ros>
-      <robotNamespace>/robotpadi</robotNamespace>
+      <robotNamespace>/polebot_land</robotNamespace>
       <topicName>/odom</topicName>
     </ros>

File: src/polebot_land/urdf/ros2_control.xacro (robot description, xacro)
@@ -28,5 +28,5 @@
    <gazebo>
       <plugin filename="gz_ros2_control-system" name="gz_ros2_control::GazeboSimROS2ControlPlugin">
-        <parameters>/home/satyo03/TA_robotpadi/install/robotpadi/share/robotpadi/config/diff_drive_controller.yaml</parameters>
+        <parameters>$(find polebot_land)/config/diff_drive_controller.yaml</parameters>
       </plugin>
   </gazebo>
